Commit message: Added libgazebo_ros_diff_drive.so and libgazebo_ros_laser.so plugins

File: my_rb1_description/urdf/my_rb1_robot.urdf (robot description, URDF)
Before this commit: robot robot, 7 links, 6 joints
Links:
- link back_caster: mass 0.5 -> 0.25
- link base_link: mass 22.0 -> 23.5
- link front_caster: mass 0.5 -> 0.25
- link left_wheel: mass 1.0 -> 0.5
- link right_wheel: mass 1.0 -> 0.5
Joints:
- joint left_wheel_joint: limit effort=10000 velocity=1000 -> effort=1000.0 velocity=1000.0
- joint right_wheel_joint: limit effort=10000 velocity=1000 -> effort=1000.0 velocity=1000.0

Commit message: amended errors in links and tuned kp kd values for robot model in Gazebo

File: my_rb1_description/urdf/my_rb1_robot.urdf (robot description, URDF)
Before this commit: robot robot, 7 links, 6 joints
Joints:
- joint back_caster_joint: axis (none) -> 1 1 0; type fixed -> continuous
- joint base_footprint_joint: child base_footprint -> base_link; origin xyz=0 0 -0.15 rpy=0 0 0 -> xyz=0 0 0.15 rpy=0 0 0; parent base_link -> base_footprint
- joint front_caster_joint: axis (none) -> 1 1 0; type fixed -> continuous

Commit message: Added laser scanner box

File: my_rb1_description/urdf/my_rb1_robot.urdf (robot description, URDF)
Before this commit: robot robot, 7 links, 6 joints
Links:
- link front_laser: geometry collision box size=0.025 0.025 0.025; visual box size=0.025 0.025 0.025

Commit message: Distributed weight of robot and added springs and dampers

File: my_rb1_description/urdf/my_rb1_robot.urdf (robot description, URDF)
Before this commit: robot robot, 7 links, 6 joints
Links:
- link base_link: mass 23.5 -> 10.0
- link left_wheel: mass 0.5 -> 7.25
- link right_wheel: mass 0.5 -> 7.25
Joints:
- joint back_caster_joint: axis 1 1 0 -> 0 1 0; origin xyz=0.1 0.0 -0.15 rpy=0 0 0 -> xyz=-0.1 0.0 -0.15 rpy=0 0 0
- joint front_caster_joint: axis 1 1 0 -> 0 1 0; origin xyz=-0.1 0.0 -0.15 rpy=0 0 0 -> xyz=0.1 0.0 -0.15 rpy=0 0 0
- joint left_wheel_joint: origin xyz=0 -0.2 -0.15 rpy=0 0 0 -> xyz=0 0.2 -0.15 rpy=0 0 0
- joint right_wheel_joint: origin xyz=0 0.2 -0.15 rpy=0 0 0 -> xyz=0 -0.2 -0.15 rpy=0 0 0

Commit message: Added correct axis to collision tags of wheels. Unpaused gazebo world in launch file

File: my_rb1_description/urdf/my_rb1_robot.urdf (robot description, URDF)
Before this commit: robot robot, 7 links, 6 joints
Links:
- link back_caster: mass 0.25 -> 0.5
- link base_link: mass 10.0 -> 5.0
- link front_caster: mass 0.25 -> 0.5
- link left_wheel: mass 7.25 -> 9.5
- link right_wheel: mass 7.25 -> 9.5
Joints:
- joint back_caster_joint: type continuous -> fixed
- joint front_caster_joint: type continuous -> fixed
